File: kicad/current_version/working/working.kicad_pcb (KiCad board)
At the start: 2 copper layers, 16 parts, among them J1 itq32at328_electronic_ic_tqfp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, J2 pms2231117, J3 scumnsmo, U1 bbat328, U2 isp16ch340c, x1 x3213mhz16

Commit message: updated gitignore
Parts:
- added C3: c6nf10, oomlout_oomp_part_footprints:c6nf10_electronic_capacitor_0603_10_nano_farad, F.Cu at (56.4, 79.2)
- added C4: c6nf100, oomlout_oomp_part_footprints:c6nf100_electronic_capacitor_0603_100_nano_farad, F.Cu at (45.2, 44.2)
- added C5: c6pf22, oomlout_oomp_part_footprints:c6pf22_electronic_capacitor_0603_22_pico_farad, F.Cu at (29.2, 46.7)
- added C6: c6pf22, oomlout_oomp_part_footprints:c6pf22_electronic_capacitor_0603_22_pico_farad, F.Cu at (27.4, 43.2)
- added C7: c6pf22, oomlout_oomp_part_footprints:c6pf22_electronic_capacitor_0603_22_pico_farad, F.Cu at (39.4, 95.5)
- added C8: c6pf22, oomlout_oomp_part_footprints:c6pf22_electronic_capacitor_0603_22_pico_farad, F.Cu at (33.5, 91.9)
- added C9: c6nf100, oomlout_oomp_part_footprints:c6nf100_electronic_capacitor_0603_100_nano_farad, F.Cu at (41.7, 50.3)
- added J4: b3560s, oomlout_oomp_part_footprints:b3560s_electronic_button_3_5_mm_x_6_mm_x_2_5_mm_surface_mount, F.Cu at (41.1, 39.1)
- added J5: hi12x3p, oomlout_oomp_part_footprints:hi12x3p_electronic_header_2d54_mm_dual_row_2x3_dual_row_6_pin, F.Cu at (39.1, 21.8)
- added nt1: nt2, oomlout_oomp_part_footprints:nt2_electronic_nettie_2_nets_smd, F.Cu at (86.9, 46.9)
- added nt2: nt2, oomlout_oomp_part_footprints:nt2_electronic_nettie_2_nets_smd, F.Cu at (86.9, 48.4)
- added nt3: nt2, oomlout_oomp_part_footprints:nt2_electronic_nettie_2_nets_smd, F.Cu at (86.9, 49.9)
- added nt4: nt2, oomlout_oomp_part_footprints:nt2_electronic_nettie_2_nets_smd, F.Cu at (86.9, 51.4)
- added nt5: nt2, oomlout_oomp_part_footprints:nt2_electronic_nettie_2_nets_smd, F.Cu at (86.9, 52.9)
- added nt6: nt2, oomlout_oomp_part_footprints:nt2_electronic_nettie_2_nets_smd, F.Cu at (86.9, 54.4)
- added x2: xcr3213mhz12, oomlout_oomp_part_footprints:xcr3213mhz12_electronic_ceramic_resonator_3213_3_pin_ground_pin_2_12_mega_hertz, F.Cu at (39.4, 90.9)
- C1, C2: value catuf4d7 -> catuf4d716v; footprint oomlout_oomp_part_footprints:catuf4d7_electronic_capacitor_3216_avx_a_tantalum_4_7_micro_farad_16_volt -> oomlout_oomp_part_footprints:catuf4d716v_electronic_capacitor_3216_avx_a_tantalum_4_7_micro_farad_16_volt
- J1: value itq32at328_electronic_ic_tqfp_32_mcu_atmega328_microchip_atmega328p_aur -> itq32at328
- J2: value pms2231117 -> pms22311171d5v; footprint oomlout_oomp_part_footprints:pms2231117_electronic_pmic_sot_223_linear_1117_5v -> oomlout_oomp_part_footprints:pms22311171d5v_electronic_pmic_sot_223_linear_1117_1_5_volt
- U2: value isp16ch340c -> isp16ch340g; footprint oomlout_oomp_part_footprints:isp16ch340c_electronic_ic_sop_16_converter_usb_to_serial_converter_wch_ch340c -> oomlout_oomp_part_footprints:isp16ch340g_electronic_ic_sop_16_converter_usb_to_serial_converter_wch_ch340g
- x1: value x3213mhz16 -> xcr3213mhz16; footprint oomlout_oomp_part_footprints:x3213mhz16_electronic_crystal_3213_3_pin_ground_pin_2_16_mega_hertz -> oomlout_oomp_part_footprints:xcr3213mhz16_electronic_ceramic_resonator_3213_3_pin_ground_pin_2_16_mega_hertz
- moved C2 45.6 mm to (30.8, 81.8)
- moved C1 44.6 mm to (31.3, 77.7)
- moved U2 40.4 mm to (47.2, 89.9)
- moved J3 38.8 mm to (42.3, 61.6)
- moved R4 38.5 mm to (46.2, 30.5), turned to 90 degrees
- moved R3 37.5 mm to (43.7, 30.5), turned to 90 degrees
- moved R1 37.1 mm to (38.1, 30.3), turned to 90 degrees
- moved R2 37.1 mm to (41.1, 30.3), turned to 90 degrees
- moved L1 33.4 mm to (38.1, 26.7), turned to 90 degrees
- moved L2 30.8 mm to (41.1, 26.6), turned to 90 degrees
- moved L3 29.0 mm to (43.7, 26.6), turned to 90 degrees
- moved x1 27.7 mm to (36.1, 45.2)
- moved L4 27.6 mm to (46.2, 26.6), turned to 90 degrees
- moved J2 21.6 mm to (45.2, 78.7)
- moved J1 19.4 mm to (41.7, 50.3), turned to 90 degrees
Connections:
- net /pb3 renamed /mosi
- net /pb4 renamed /miso
- net /pc4 renamed /adc4
- net /pc5 renamed /adc5
- C2 pad 1: +3V3 -> +5V
- J2 pad 2: +3V3 -> +5V
- J3 pad 6: /usb_shield -> GND
- U2 pad 2: /pd0 -> /tx_ch340
- U2 pad 3: /pd1 -> /rx_ch340
- U2 pad 4: unconnected-(U2-V3-Pad4) -> Net-(U2-V3)
- U2 pad 7: unconnected-(U2-NC-Pad7) -> /xtal_1_ch340
- U2 pad 8: unconnected-(U2-NC-Pad8) -> /xtal_2_ch340
- x1 pad 1: /pb6 -> /xtal_1
- x1 pad 3: /pb7 -> /xtal_2

Commit message: workings
Parts:
- removed C4: c6nf100, oomlout_oomp_part_footprints:c6nf100_electronic_capacitor_0603_100_nano_farad
- removed C8: c6pf22, oomlout_oomp_part_footprints:c6pf22_electronic_capacitor_0603_22_pico_farad
- removed J4: b3560s, oomlout_oomp_part_footprints:b3560s_electronic_button_3_5_mm_x_6_mm_x_2_5_mm_surface_mount
- removed J5: hi12x3p, oomlout_oomp_part_footprints:hi12x3p_electronic_header_2d54_mm_dual_row_2x3_dual_row_6_pin
- removed L1, L2, L3, L4: l6r, oomlout_oomp_part_footprints:l6r_electronic_led_0603_red
- removed nt3, nt4: nt2, oomlout_oomp_part_footprints:nt2_electronic_nettie_2_nets_smd
- removed x1: xcr3213mhz16, oomlout_oomp_part_footprints:xcr3213mhz16_electronic_ceramic_resonator_3213_3_pin_ground_pin_2_16_mega_hertz
- removed x2: xcr3213mhz12, oomlout_oomp_part_footprints:xcr3213mhz12_electronic_ceramic_resonator_3213_3_pin_ground_pin_2_12_mega_hertz
- added 1111: nt2, oomlout_oomp_part_footprints:nt2_electronic_nettie_2_nets_smd, F.Cu at (67.7, 42.5)
- added 11111: nt2, oomlout_oomp_part_footprints:nt2_electronic_nettie_2_nets_smd, F.Cu at (67.7, 44.0)
- added B1: b3560s, oomlout_oomp_part_footprints:b3560s_electronic_button_3_5_mm_x_6_mm_x_2_5_mm_surface_mount, F.Cu at (52.4, 66.0)
- added D1: dssod123pmb2, oomlout_oomp_part_footprints:dssod123pmb2_electronic_diode_schottky_sod_123_package_marking_b2_mbr0520, F.Cu at (62.9, 37.9)
- added L1_RX1: l6r, oomlout_oomp_part_footprints:l6r_electronic_led_0603_red, F.Cu at (59.8, 64.7)
- added L2_TX1: l6r, oomlout_oomp_part_footprints:l6r_electronic_led_0603_red, F.Cu at (59.8, 67.3)
- added L3_POW1: l6r, oomlout_oomp_part_footprints:l6r_electronic_led_0603_red, F.Cu at (59.8, 69.9)
- added L4_L1: l6r, oomlout_oomp_part_footprints:l6r_electronic_led_0603_red, F.Cu at (59.8, 72.5)
- added R5: r6o102, oomlout_oomp_part_footprints:r6o102_electronic_resistor_0603_1000_ohm, F.Cu at (57.2, 45.5)
- added R6: r6o102, oomlout_oomp_part_footprints:r6o102_electronic_resistor_0603_1000_ohm, F.Cu at (57.2, 48.0)
- added R7: r6o102, oomlout_oomp_part_footprints:r6o102_electronic_resistor_0603_1000_ohm, F.Cu at (57.2, 50.5)
- added U3: isp16ch340g, oomlout_oomp_part_footprints:isp16ch340g_electronic_ic_sop_16_converter_usb_to_serial_converter_wch_ch340g, F.Cu at (63.1, 57.5)
- added X1: xcr3213mhz16, oomlout_oomp_part_footprints:xcr3213mhz16_electronic_ceramic_resonator_3213_3_pin_ground_pin_2_16_mega_hertz, F.Cu at (64.3, 65.2)
- added X2: xcr3213mhz12, oomlout_oomp_part_footprints:xcr3213mhz12_electronic_ceramic_resonator_3213_3_pin_ground_pin_2_12_mega_hertz, F.Cu at (64.3, 69.1)
- C5, C6, C7: value c6pf22 -> c6nf100; footprint oomlout_oomp_part_footprints:c6pf22_electronic_capacitor_0603_22_pico_farad -> oomlout_oomp_part_footprints:c6nf100_electronic_capacitor_0603_100_nano_farad
- J1: value itq32at328 -> bbat328; footprint oomlout_oomp_part_footprints:itq32at328_electronic_ic_tqfp_32_mcu_atmega328_microchip_atmega328p_aur -> oomlout_oomp_part_footprints:bbat328_electronic_breakout_board_mcu_atmega328_shennie
- J2: value pms22311171d5v -> hi12x3p; footprint oomlout_oomp_part_footprints:pms22311171d5v_electronic_pmic_sot_223_linear_1117_1_5_volt -> oomlout_oomp_part_footprints:hi12x3p_electronic_header_2d54_mm_dual_row_2x3_dual_row_6_pin
- U1: value bbat328 -> itq32at328; footprint oomlout_oomp_part_footprints:bbat328_electronic_breakout_board_mcu_atmega328_shennie -> oomlout_oomp_part_footprints:itq32at328_electronic_ic_tqfp_32_mcu_atmega328_microchip_atmega328p_aur
- U2: value isp16ch340g -> pms22311171d5v; footprint oomlout_oomp_part_footprints:isp16ch340g_electronic_ic_sop_16_converter_usb_to_serial_converter_wch_ch340g -> oomlout_oomp_part_footprints:pms22311171d5v_electronic_pmic_sot_223_linear_1117_1_5_volt
- moved C2 57.0 mm to (62.9, 34.6)
- moved C1 56.0 mm to (62.9, 31.5)
- moved U1 46.8 mm to (0.00, -6.05)
- moved C7 46.1 mm to (49.2, 50.5)
- moved J2 38.3 mm to (61.5, 44.0)
- moved C3 37.0 mm to (49.2, 43.0)
- moved J3 29.1 mm to (53.6, 34.8)
- moved C6 22.3 mm to (49.2, 48.0)
- moved R3 22.2 mm to (53.2, 50.5), turned to 0 degrees
- moved R1 21.4 mm to (53.2, 45.5), turned to 0 degrees
- moved R2 21.4 mm to (53.2, 48.0), turned to 0 degrees
- moved C5 20.0 mm to (49.2, 45.5)
- moved nt5 19.7 mm to (67.7, 48.5)
- moved nt6 19.7 mm to (67.7, 50.0)
- moved J1 19.7 mm to (29.9, 34.5), turned to 0 degrees
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Connections:
- net /led_4 renamed /d13
- C1 pad 2: GND -> +5V
- C2 pad 2: GND -> +5V
- C3 pad 1: Net-(U2-V3) -> Net-(U3-V3)
- C3 pad 2: GND -> +5V
- C5 pad 1: /xtal_1 -> +5V
- C5 pad 2: GND -> /pc6
- C6 pad 1: /xtal_2 -> +5V
- C6 pad 2: GND -> +5V
- C7 pad 1: /xtal_1_ch340 -> +12V
- C7 pad 2: GND -> +5V
- C9 pad 2: GND -> +5V
- J1 pad 1: /pd3 -> /pd1
- J1 pad 10: /pd6 -> /pd7
- J1 pad 11: /pd7 -> /pb0
- J1 pad 12: /pb0 -> /pb1
- J1 pad 13: /pb1 -> /pb2
- J1 pad 14: /pb2 -> /mosi
- J1 pad 15: /mosi -> /miso
- J1 pad 16: /miso -> /pb5
- J1 pad 17: /pb5 -> +3V3
- J1 pad 18: +5V -> /aref
- J1 pad 19: /adc6 -> /pc0
- J1 pad 2: /pd4 -> /pd0
- J1 pad 20: /aref -> /pc1
- J1 pad 21: GND -> /pc2
- J1 pad 22: /adc7 -> /pc3
- J1 pad 23: /pc0 -> /adc4
- J1 pad 24: /pc1 -> /adc5
- J1 pad 25: /pc2 -> /adc6
- J1 pad 26: /pc3 -> /adc7
- J1 pad 27: /adc4 -> +5V
- J1 pad 28: /adc5 -> /pc6
- J1 pad 29: /pc6 -> +5V
- J1 pad 3: GND -> /pc6
- J1 pad 30: /pd0 -> +12V
- J1 pad 5: GND -> /pd2
- J1 pad 6: +5V -> /pd3
- J1 pad 7: /pb6 -> /pd4
- J1 pad 8: /pb7 -> /pd5
- J1 pad 9: /pd5 -> /pd6
- J2 pad 1: GND -> unconnected-(J2-Pin_1-Pad1)
- J2 pad 3: +12V -> unconnected-(J2-Pin_3-Pad3)
- J2 pad 4: (no net) -> /mosi
- J3 pad 1: +5V -> Net-(D1-A)
- J3 pad 5: GND -> +5V
- J3 pad 6: GND -> +5V
- R1 pad 2: /led_1 -> /pd0
- R2 pad 2: /led_2 -> /pd1
- R3 pad 2: /led_3 -> +5V
- U1 pad 1: /pd1 -> /pd3
- U1 pad 10: /pd7 -> /pd6
- U1 pad 11: /pb0 -> /pd7
- U1 pad 12: /pb1 -> /pb0
- U1 pad 13: /pb2 -> /pb1
- U1 pad 14: /mosi -> /pb2
- U1 pad 15: /miso -> /mosi
- U1 pad 16: /pb5 -> /miso
- U1 pad 17: +3V3 -> /pb5
- U1 pad 18: /aref -> +5V
- U1 pad 19: /pc0 -> /adc6
- U1 pad 2: /pd0 -> /pd4
- U1 pad 20: /pc1 -> /aref
- U1 pad 21: /pc2 -> +5V
- U1 pad 22: /pc3 -> /adc7
- U1 pad 23: /adc4 -> /pc0
- U1 pad 24: /adc5 -> /pc1
- U1 pad 25: /adc6 -> /pc2
- U1 pad 26: /adc7 -> /pc3
- U1 pad 27: +5V -> /adc4
- U1 pad 28: /pc6 -> /adc5
- U1 pad 29: GND -> /pc6
- U1 pad 3: /pc6 -> +5V
- U1 pad 30: +12V -> /pd0
- U1 pad 4: GND -> +5V
- U1 pad 5: /pd2 -> +5V
- U1 pad 6: /pd3 -> +5V
- U1 pad 7: /pd4 -> /pb6
- U1 pad 8: /pd5 -> /pb7
- U1 pad 9: /pd6 -> /pd5
- U2 pad 1: GND -> +5V
- U2 pad 2: /tx_ch340 -> +5V
- U2 pad 3: /rx_ch340 -> +12V
- U2 pad 4: Net-(U2-V3) -> (no net)

Commit message: workings
Parts:
- removed C9: c6nf100, oomlout_oomp_part_footprints:c6nf100_electronic_capacitor_0603_100_nano_farad
- added C4: c6nf100, oomlout_oomp_part_footprints:c6nf100_electronic_capacitor_0603_100_nano_farad, B.Cu at (54.1, 53.3)
- C1, C2, C3, C5, C6, C7, D1, R5, R6, R7, U2, U3, X2: moved to B.Cu
- moved U2 55.7 mm to (107.6, 68.1), turned to 180 degrees
- moved C3 47.3 mm to (94.5, 29.5), turned to 180 degrees
- moved C5 42.7 mm to (90.9, 36.6), turned to 180 degrees
- moved C6 42.7 mm to (90.9, 39.1), turned to 180 degrees
- moved C7 42.7 mm to (90.9, 41.6), turned to 180 degrees
- moved C1 41.6 mm to (104.4, 32.7), turned to 180 degrees
- moved C2 41.6 mm to (104.4, 35.9), turned to 180 degrees
- moved D1 41.5 mm to (104.4, 39.1), turned to 180 degrees
- moved U3 33.7 mm to (96.4, 52.3), turned to 180 degrees
- moved X2 31.3 mm to (95.2, 63.9), turned to 180 degrees
- moved R5 27.2 mm to (82.9, 36.6), turned to 180 degrees
- moved R6 27.2 mm to (82.9, 39.1), turned to 180 degrees
- moved R7 27.2 mm to (82.9, 41.6), turned to 180 degrees
- moved R3 26.3 mm to (74.9, 35.6)
- moved R2 20.5 mm to (69.1, 35.0)
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Connections:
- net /pc0 renamed /adc0
- net /pc1 renamed /adc1
- net /pc2 renamed /adc2
- net /pc3 renamed /adc3
- B1 pad 2: +5V -> GND
- C1 pad 2: +5V -> GND
- C2 pad 2: +5V -> GND
- C3 pad 2: +5V -> GND
- C6 pad 2: +5V -> GND
- C7 pad 2: +5V -> GND
- J1 pad 29: +5V -> GND
- J1 pad 4: +5V -> GND
- J2 pad 1: unconnected-(J2-Pin_1-Pad1) -> /miso
- J2 pad 3: unconnected-(J2-Pin_3-Pad3) -> /pb5
- J2 pad 5: unconnected-(J2-Pin_5-Pad5) -> /pc6
- J2 pad 6: +5V -> GND
- J3 pad 5: +5V -> GND
- J3 pad 6: +5V -> GND
- L3_POW1 pad 1: +5V -> GND
- L4_L1 pad 1: +5V -> GND
- U1 pad 21: +5V -> GND
- U1 pad 3: +5V -> GND
- U1 pad 5: +5V -> GND
- U2 pad 1: +5V -> GND
- U3 pad 1: +5V -> GND
- U3 pad 7: /xtal_1 -> /xtal1_ch340
- U3 pad 8: /xtal_2 -> /xtal2_ch340
- X1 pad 1: /xtal_1_atmega328 -> /pb6
- X1 pad 2: +5V -> GND
- X1 pad 3: /xtal_2_atmega328 -> /pb7
- X2 pad 1: /xtal_1_ch340 -> /xtal1_ch340
- X2 pad 2: +5V -> GND
- X2 pad 3: /xtal_2_ch340 -> /xtal2_ch340
