File: kicad/current_version/working/working.kicad_sch (KiCad schematic)
At the start: 32 parts, among them J1 itq32at328, J2 b3560s, J2 pms22311171d5v, J3 scumnsmo, J5 hi12x3p, U1 bbat328, U1 isp16ch340g, x1 xcr3213mhz12, x1 xcr3213mhz16

Commit message: updated gitignore
Parts:
- 111, 1111, nt1, nt2, nt3, nt4: footprint oomlout_oomp_part_footprints:nt2_electronic_nettie_2_nets_smd -> oomlout_oomp_part_kicad_footprints:nt2_electronic_nettie_2_nets_smd
- C1, C2: footprint oomlout_oomp_part_footprints:c6pf22_electronic_capacitor_0603_22_pico_farad -> oomlout_oomp_part_kicad_footprints:c6pf22_electronic_capacitor_0603_22_pico_farad
- C1, C2: footprint oomlout_oomp_part_footprints:catuf4d716v_electronic_capacitor_3216_avx_a_tantalum_4_7_micro_farad_16_volt -> oomlout_oomp_part_kicad_footprints:catuf4d716v_electronic_capacitor_3216_avx_a_tantalum_4_7_micro_farad_16_volt
- C1: footprint oomlout_oomp_part_footprints:c6nf100_electronic_capacitor_0603_100_nano_farad -> oomlout_oomp_part_kicad_footprints:c6nf100_electronic_capacitor_0603_100_nano_farad
- C2: footprint oomlout_oomp_part_footprints:c6nf10_electronic_capacitor_0603_10_nano_farad -> oomlout_oomp_part_kicad_footprints:c6nf10_electronic_capacitor_0603_10_nano_farad
- J2: renamed from J5; footprint oomlout_oomp_part_footprints:hi12x3p_electronic_header_2d54_mm_dual_row_2x3_dual_row_6_pin -> oomlout_oomp_part_kicad_footprints:hi12x3p_electronic_header_2d54_mm_dual_row_2x3_dual_row_6_pin
- J2: footprint oomlout_oomp_part_footprints:b3560s_electronic_button_3_5_mm_x_6_mm_x_2_5_mm_surface_mount -> oomlout_oomp_part_kicad_footprints:b3560s_electronic_button_3_5_mm_x_6_mm_x_2_5_mm_surface_mount
- J3: footprint oomlout_oomp_part_footprints:scumnsmo_electronic_socket_usb_mini_surface_mount_only -> oomlout_oomp_part_kicad_footprints:scumnsmo_electronic_socket_usb_mini_surface_mount_only
- L1, L2, L3, L4: footprint oomlout_oomp_part_footprints:l6r_electronic_led_0603_red -> oomlout_oomp_part_kicad_footprints:l6r_electronic_led_0603_red
- R1, R2, R3, R4: footprint oomlout_oomp_part_footprints:r6o102_electronic_resistor_0603_1000_ohm -> oomlout_oomp_part_kicad_footprints:r6o102_electronic_resistor_0603_1000_ohm
- U1: renamed from J1; footprint oomlout_oomp_part_footprints:itq32at328_electronic_ic_tqfp_32_mcu_atmega328_microchip_atmega328p_aur -> oomlout_oomp_part_kicad_footprints:itq32at328_electronic_ic_tqfp_32_mcu_atmega328_microchip_atmega328p_aur
- U1: footprint oomlout_oomp_part_footprints:isp16ch340g_electronic_ic_sop_16_converter_usb_to_serial_converter_wch_ch340g -> oomlout_oomp_part_kicad_footprints:isp16ch340g_electronic_ic_sop_16_converter_usb_to_serial_converter_wch_ch340g
- U2: renamed from J2; footprint oomlout_oomp_part_footprints:pms22311171d5v_electronic_pmic_sot_223_linear_1117_1_5_volt -> oomlout_oomp_part_kicad_footprints:pms22311171d5v_electronic_pmic_sot_223_linear_1117_1_5_volt
- x1: footprint oomlout_oomp_part_footprints:xcr3213mhz12_electronic_ceramic_resonator_3213_3_pin_ground_pin_2_12_mega_hertz -> oomlout_oomp_part_kicad_footprints:xcr3213mhz12_electronic_ceramic_resonator_3213_3_pin_ground_pin_2_12_mega_hertz
- x1: footprint oomlout_oomp_part_footprints:xcr3213mhz16_electronic_ceramic_resonator_3213_3_pin_ground_pin_2_16_mega_hertz -> oomlout_oomp_part_kicad_footprints:xcr3213mhz16_electronic_ceramic_resonator_3213_3_pin_ground_pin_2_16_mega_hertz

Commit message: workings
Parts:
- removed C1 (x2), C2 (x2): c6pf22, oomlout_oomp_part_kicad_footprints:c6pf22_electronic_capacitor_0603_22_pico_farad, symbol oomlout_oomp_part_symbols:c6pf22_electronic_capacitor_0603_22_pico_farad
- removed L1, L2, L3, L4: l6r, oomlout_oomp_part_kicad_footprints:l6r_electronic_led_0603_red, symbol oomlout_oomp_part_symbols:l6r_electronic_led_0603_red
- removed R1, R2, R3, R4: r6o102, oomlout_oomp_part_kicad_footprints:r6o102_electronic_resistor_0603_1000_ohm, symbol oomlout_oomp_part_symbols:r6o102_electronic_resistor_0603_1000_ohm
- removed nt3, nt4: nt2, oomlout_oomp_part_kicad_footprints:nt2_electronic_nettie_2_nets_smd, symbol oomlout_oomp_part_symbols:nt2_electronic_nettie_2_nets_smd
- added 11, 111: nt2, nt2_electronic_nettie_2_nets_smd, symbol oomlout_oomp_part_symbols:nt2_electronic_nettie_2_nets_smd
- added C6, C7: c6nf100, oomlout_oomp_part_footprints:c6nf100_electronic_capacitor_0603_100_nano_farad, symbol oomlout_oomp_part_symbols:c6nf100_electronic_capacitor_0603_100_nano_farad
- added D1: dssod123pmb2, oomlout_oomp_part_footprints:dssod123pmb2_electronic_diode_schottky_sod_123_package_marking_b2_mbr0520, symbol oomlout_oomp_part_symbols:dssod123pmb2_electronic_diode_schottky_sod_123_packag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
- added L1 (x2), L2 (x2): l6r, l6r_electronic_led_0603_red, symbol oomlout_oomp_part_symbols:l6r_electronic_led_0603_red
- added R1 (x2), R2: r6o102, oomlout_oomp_part_footprints:r6o102_electronic_resistor_0603_1000_ohm, symbol oomlout_oomp_part_symbols:r6o102_electronic_resistor_0603_1000_ohm
- added R1 (x2), R2 (x2): r6o102, r6o102_electronic_resistor_0603_1000_ohm, symbol oomlout_oomp_part_symbols:r6o102_electronic_resistor_0603_1000_ohm
- C1: footprint oomlout_oomp_part_kicad_footprints:c6nf100_electronic_capacitor_0603_100_nano_farad -> oomlout_oomp_part_footprints:c6nf100_electronic_capacitor_0603_100_nano_farad
- C2: footprint oomlout_oomp_part_kicad_footprints:c6nf10_electronic_capacitor_0603_10_nano_farad -> c6nf10_electronic_capacitor_0603_10_nano_farad
- U1: footprint oomlout_oomp_part_kicad_footprints:isp16ch340g_electronic_ic_sop_16_converter_usb_to_serial_converter_wch_ch340g -> isp16ch340g_electronic_ic_sop_16_converter_usb_to_serial_converter_wch_ch340g
Connections:
- net +12V: now also C7.1
- net +5V: now also C1.2, C1.2, C2.2, C2.2, J2.2, J2.6 (Pin_6), J3.5 (GND), J3.6 (Shield), U1.1 (GND), U1.21 (GND), U1.29 (GND), U1.3 (GND), U1.4 (GND), U1.5 (GND), U2.1 (GND), x1.2, x1.2, C6.1, C6.2, C7.2, D1.1 (K), L1.1 (K), L1.2 (A), L2.1 (K), L2.2 (A), R1.2, R1.2; no longer J3.1 (VBUS)
- net dtr: now also R1.1
- net pc6: now also C1.2
- net pd0: now also 11.2, R2.2
- net pd1: now also 111.2, R1.2
- net rx_ch340: now also 111.1, R2.2; no longer U1.3 (RXD)
- net tx_ch340: now also 11.1, R1.2; no longer U1.2 (TXD)
- net xtal_1: now also U1.7 (XI); no longer x1.1
- net xtal_1_ch340: no longer U1.7 (XI)
- net xtal_2: now also U1.8 (XO); no longer x1.3
- net xtal_2_ch340: no longer U1.8 (XO)
- removed net GND: C1.2, C1.2, C1.2, C2.2, C2.2, J2.2, J2.6 (Pin_6), J3.5 (GND), J3.6 (Shield), U1.1 (GND), U1.21 (GND), U1.29 (GND), U1.3 (GND), U1.4 (GND), U1.5 (GND), U2.1 (GND), x1.2, x1.2
- new net: R1.1, U1.2 (TXD)
- new net: L2.1 (K), R2.1
- new net: L2.2 (A), R2.1
- new net: D1.2 (A), J3.1 (VBUS)
- new net: L1.1 (K), R1.1
- new net: L1.2 (A), R1.1
- new net: R2.1, U1.3 (RXD)
- new net d13: R2.2
- new net xtal_1_atmega328: x1.1
- new net xtal_2_atmega328: x1.3
Other:
- note added: "auto_reset"
- note added: "ch340328_tx_rx_patch_block"
- note added: "module connector usb_mini surface_mount_only back_power_protected"
- note added: "oomp ic usb_to_serial_bridge sop_16 5_volt ch340g"
- note added: "oomp led 0603 red two_leds common_ground"
- note added: "oomp led 0603 red two_leds common_supply"
- note added: "oomp logic arduino_compatible auto_reset_circuit"
- note added: "xcr_atmega328"
- note removed: "module connector usb_mini surface_mount_only"
- note removed: "oomp led 0603 red four_leds"
- note removed: "oomp sop_16 usb_to_serial_bridge 5_volt ch340g"
- note removed: "xcr"
- moved on the sheet: 111, 1111, U1

Commit message: workings
Parts:
- 11, 111: footprint nt2_electronic_nettie_2_nets_smd -> oomlout_oomp_part_footprints:nt2_electronic_nettie_2_nets_smd
- 111, 1111, nt1, nt2: footprint oomlout_oomp_part_kicad_footprints:nt2_electronic_nettie_2_nets_smd -> oomlout_oomp_part_footprints:nt2_electronic_nettie_2_nets_smd
- C1, C2: footprint oomlout_oomp_part_kicad_footprints:catuf4d716v_electronic_capacitor_3216_avx_a_tantalum_4_7_micro_farad_16_volt -> oomlout_oomp_part_footprints:catuf4d716v_electronic_capacitor_3216_avx_a_tantalum_4_7_micro_farad_16_volt
- C1: footprint oomlout_oomp_part_kicad_footprints:c6nf100_electronic_capacitor_0603_100_nano_farad -> oomlout_oomp_part_footprints:c6nf100_electronic_capacitor_0603_100_nano_farad
- C2: footprint c6nf10_electronic_capacitor_0603_10_nano_farad -> oomlout_oomp_part_footprints:c6nf10_electronic_capacitor_0603_10_nano_farad
- J2: footprint oomlout_oomp_part_kicad_footprints:hi12x3p_electronic_header_2d54_mm_dual_row_2x3_dual_row_6_pin -> oomlout_oomp_part_footprints:hi12x3p_electronic_header_2d54_mm_dual_row_2x3_dual_row_6_pin
- J2: footprint oomlout_oomp_part_kicad_footprints:b3560s_electronic_button_3_5_mm_x_6_mm_x_2_5_mm_surface_mount -> oomlout_oomp_part_footprints:b3560s_electronic_button_3_5_mm_x_6_mm_x_2_5_mm_surface_mount
- J3: footprint oomlout_oomp_part_kicad_footprints:scumnsmo_electronic_socket_usb_mini_surface_mount_only -> oomlout_oomp_part_footprints:scumnsmo_electronic_socket_usb_mini_surface_mount_only
- L1, L2: footprint l6r_electronic_led_0603_red -> oomlout_oomp_part_footprints:l6r_electronic_led_0603_red
- R1, R2: footprint r6o102_electronic_resistor_0603_1000_ohm -> oomlout_oomp_part_footprints:r6o102_electronic_resistor_0603_1000_ohm
- U1: footprint oomlout_oomp_part_kicad_footprints:itq32at328_electronic_ic_tqfp_32_mcu_atmega328_microchip_atmega328p_aur -> oomlout_oomp_part_footprints:itq32at328_electronic_ic_tqfp_32_mcu_atmega328_microchip_atmega328p_aur
- U1: footprint isp16ch340g_electronic_ic_sop_16_converter_usb_to_serial_converter_wch_ch340g -> oomlout_oomp_part_footprints:isp16ch340g_electronic_ic_sop_16_converter_usb_to_serial_converter_wch_ch340g
- U2: footprint oomlout_oomp_part_kicad_footprints:pms22311171d5v_electronic_pmic_sot_223_linear_1117_1_5_volt -> oomlout_oomp_part_footprints:pms22311171d5v_electronic_pmic_sot_223_linear_1117_1_5_volt
- x1: footprint oomlout_oomp_part_kicad_footprints:xcr3213mhz12_electronic_ceramic_resonator_3213_3_pin_ground_pin_2_12_mega_hertz -> oomlout_oomp_part_footprints:xcr3213mhz12_electronic_ceramic_resonator_3213_3_pin_ground_pin_2_12_mega_hertz
- x1: footprint oomlout_oomp_part_kicad_footprints:xcr3213mhz16_electronic_ceramic_resonator_3213_3_pin_ground_pin_2_16_mega_hertz -> oomlout_oomp_part_footprints:xcr3213mhz16_electronic_ceramic_resonator_3213_3_pin_ground_pin_2_16_mega_hertz

Commit message: workings
Connections:
- net pc0 is gone; now on net adc0: U1.19 (A0), U1.23 (PC0)
- net pc1 is gone; now on net adc1: U1.20 (A1), U1.24 (PC1)
- net pc2 is gone; now on net adc2: U1.21 (A2), U1.25 (PC2)
- net pc3 is gone; now on net adc3: U1.22 (A3), U1.26 (PC3)
- net xtal_1_atmega328 is gone; now on net pb6: x1.1
- net xtal_1_ch340 is gone; now on net xtal1_ch340: x1.1
- net xtal_2_atmega328 is gone; now on net pb7: x1.3
- net xtal_2_ch340 is gone; now on net xtal2_ch340: x1.3
- net +5V: no longer C1.2, C1.2, C2.2, C2.2, C6.2, C7.2, J2.2, J2.6 (Pin_6), J3.5 (GND), J3.6 (Shield), L1.1 (K), L2.1 (K), U1.1 (GND), U1.21 (GND), U1.29 (GND), U1.3 (GND), U1.4 (GND), U1.5 (GND), U2.1 (GND), x1.2, x1.2
- net miso: now also J2.1 (Pin_1)
- net pb5: now also J2.3 (Pin_3)
- net pc6: now also J2.5 (Pin_5)
- net xtal_1 renamed xtal1_ch340
- net xtal_2 renamed xtal2_ch340
- new net GND: C1.2, C1.2, C2.2, C2.2, C6.2, C7.2, J2.2, J2.6 (Pin_6), J3.5 (GND), J3.6 (Shield), L1.1 (K), L2.1 (K), U1.1 (GND), U1.21 (GND), U1.29 (GND), U1.3 (GND), U1.4 (GND), U1.5 (GND), U2.1 (GND), x1.2, x1.2
Changed lines of the file:
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@@
 (kicad_sch (version 20230121) (generator eeschema)
   (paper "A3")
-  (junction (at 240.03 109.22) (diameter 0) (color 0 0 0 0)
-  )
   (junction (at 312.42 107.95) (diameter 0) (color 0 0 0 0)
   )
@@
     (stroke (width 0) (type default))
   )
+  (wire (pts (xy 165.1 172.72) (xy 167.64 172.72))
+    (stroke (width 0) (type default))
+  )
   (wire (pts (xy 240.03 96.52) (xy 240.03 102.87))
     (stroke (width 0) (type default))
   )
-  (wire (pts (xy 218.44 109.22) (xy 240.03 109.22))
-    (stroke (width 0) (type default))
-  )
   (wire (pts (xy 375.92 59.69) (xy 375.92 62.23))
     (stroke (width 0) (type default))
@@
     (stroke (width 0) (type default))
   )
-  (wire (pts (xy 119.38 102.87) (xy 121.92 102.87))
+  (wire (pts (xy 119.38 102.87) (xy 127 102.87))
     (stroke (width 0) (type default))
   )
@@
     (stroke (width 0) (type default))
   )
-  (wire (pts (xy 240.03 109.22) (xy 240.03 111.76))
+  (wire (pts (xy 240.03 102.87) (xy 240.03 111.76))
     (stroke (width 0) (type default))
   )
@@
     (stroke (width 0) (type default))
   )
-  (wire (pts (xy 240.03 102.87) (xy 240.03 109.22))
-    (stroke (width 0) (type default))
-  )
   (wire (pts (xy 381 90.17) (xy 383.54 90.17))
     (stroke (width 0) (type default))
@@
     (stroke (width 0) (type default))
   )
-  (wire (pts (xy 119.38 105.41) (xy 121.92 105.41))
+  (wire (pts (xy 119.38 105.41) (xy 127 105.41))
     (stroke (width 0) (type default))
   )
@@
     (stroke (width 0) (type default))
   )
+  (wire (pts (xy 165.1 175.26) (xy 167.64 175.26))
+    (stroke (width 0) (type default))
+  )
   (wire (pts (xy 353.06 105.41) (xy 355.6 105.41))
     (stroke (width 0) (type default))
@@
     (stroke (width 0) (type default))
   )
-  (wire (pts (xy 119.38 107.95) (xy 121.92 107.95))
+  (wire (pts (xy 119.38 107.95) (xy 127 107.95))
     (stroke (width 0) (type default))
   )
@@
     (stroke (width 0) (type default))
   )
-  (wire (pts (xy 119.38 100.33) (xy 121.92 100.33))
+  (wire (pts (xy 119.38 100.33) (xy 127 100.33))
     (stroke (width 0) (type default))
   )
@@
   )
   (wire (pts (xy 381 97.79) (xy 383.54 97.79))
+    (stroke (width 0) (type default))
+  )
+  (wire (pts (xy 165.1 170.18) (xy 167.64 170.18))
     (stroke (width 0) (type default))
   )
@@
     (effects (font (size 1.27 1.27)) (justify right bottom))
   )
-  (label "xtal_1_atmega328" (at 161.29 116.84 180) (fields_autoplaced)
+  (label "xtal1_atmega328" (at 161.29 116.84 180) (fields_autoplaced)
     (effects (font (size 1.27 1.27)) (justify right bottom))
   )
@@
     (effects (font (size 1.27 1.27)) (justify right bottom))
   )
-  (label "xtal_1_ch340" (at 224.79 194.31 180) (fields_autoplaced)
+  (label "xtal1_ch340" (at 224.79 194.31 180) (fields_autoplaced)
     (effects (font (size 1.27 1.27)) (justify right bottom))
   )
@@
     (effects (font (size 1.27 1.27)) (justify left bottom))
   )
-  (label "xtal_2_ch340" (at 250.19 194.31 0) (fields_autoplaced)
+  (label "xtal2_ch340" (at 250.19 194.31 0) (fields_autoplaced)
     (effects (font (size 1.27 1.27)) (justify left bottom))
   )
@@
     (effects (font (size 1.27 1.27)) (justify left bottom))
   )
-  (label "xtal_2_atmega328" (at 186.69 116.84 0) (fields_autoplaced)
+  (label "xtal2_atmega328" (at 186.69 116.84 0) (fields_autoplaced)
     (effects (font (size 1.27 1.27)) (justify left bottom))
   )
@@
     (effects (font (size 1.27 1.27)) (justify left bottom))
   )
-  (label "xtal_1" (at 227.33 86.36 180) (fields_autoplaced)
+  (label "xtal1_ch340" (at 227.33 86.36 180) (fields_autoplaced)
     (effects (font (size 1.27 1.27)) (justify right bottom))
   )
@@
     (effects (font (size 1.27 1.27)) (justify right bottom))
   )
-  (label "xtal_2" (at 227.33 91.44 180) (fields_autoplaced)
+  (label "xtal2_ch340" (at 227.33 91.44 180) (fields_autoplaced)
     (effects (font (size 1.27 1.27)) (justify right bottom))
   )
@@
         (path "/b2804c28-0f7b-4aef-9942-b5794639a3dd"
           (reference "#PWR?") (unit 1)
-        )
-      )
-    )
-  )
-  (symbol (lib_id "power:+5V") (at 218.44 109.22 90) (unit 1)
-    (in_bom yes) (on_board yes) (dnp no) (fields_autoplaced)
-    (property "Reference" "#PWR01" (at 222.25 109.22 0)
-      (effects (font (size 1.27 1.27)) hide)
-    )
-    (property "Value" "+5V" (at 214.63 109.22 90)
-      (effects (font (size 1.27 1.27)) (justify left))
-    )
-    (property "Footprint" "" (at 218.44 109.22 0)
-      (effects (font (size 1.27 1.27)) hide)
-    )
-    (property "Datasheet" "" (at 218.44 109.22 0)
-      (effects (font (size 1.27 1.27)) hide)
-    )
-    (pin "1")
-    (instances
-      (project "working"
-        (path "/12ef09fc-ac25-49d7-9ff1-a1bc8f30d19c"
-          (reference "#PWR01") (unit 1)
-        )
-      )
-      (project "working"
-        (path "/5407c114-4107-4d84-8382-1717fb9d687c"
-          (reference "#PWR011") (unit 1)
         )
       )
@@
       (project "working"
         (path "/5407c114-4107-4d84-8382-1717fb9d687c"
-          (reference "C9") (unit 1)
-        )
-      )
+          (reference "C4") (unit 1)
+        )
+      )
