File: kicad/v_1/working/working.kicad_sch (KiCad schematic)
At the start: 28 parts, among them J2 b3560s, J2 hi12x3p, J3 scumnsmo, U1 bbat328, U1 isp16ch340g, U1 itq32at328, U2 pms22311171d5v, x1 xcr3213mhz12, x1 xcr3213mhz16

Commit message: started routing backside needs swapping over
Parts:
- added 11, 111 (x2), 1111, nt1, nt2: nt2, oomlout_oomp_part_footprints:nt2_electronic_nettie_2_nets_smd, symbol oomlout_oomp_part_symbols:nt2_electronic_nettie_2_nets_smd
Connections:
- net pd0: now also 11.2, 1111.1, 1111.2, nt2.1; no longer R1.2
- net pd1: now also 111.1, 111.2, 111.2, nt1.1; no longer R2.2
- new net rx_ch340: 111.1, R2.2, nt1.2
- new net tx_ch340: 11.1, R1.2, nt2.2
